File: bass#.kicad_sch (KiCad schematic)
At the start: 53 parts, among them J1 Trigger, J3 Output, J4 CV, Q1 2N3904, Q2 2N3904, Q3 2N3906, Q4 2N3906, U1 TL072, U2 LM13700

Commit message: trying simulation
Parts:
- added C1: 100nF, symbol Device:C
- added R2: 1M, symbol Device:R
- C4: value 2.2uF -> 2.2u
- renumbered C15 to C10, C16 to C11, C1 to C2, C2 to C3, C3 to C5, C12 to C6, C11 to C7, C13 to C8, C14 to C9, D2 to D1, D3 to D2, D1 to D3, D6 to D5, D5 to D6, J4 to J2, R3 to R1, R12 to R11, R6 to R12, R11 to R13, R13 to R14, R18 to R15, R14 to R16, R15 to R17, R19 to R18, R16 to R19, R17 to R20, R20 to R21, R2 to R3, R1 to R4, R7 to R5, R8 to R6, R5 to R7, R4 to R8
Connections:
- net GND: now also C1.1, R2.1; no longer C2.2, ImpactTone1.1, R1.2, U1.3 (+)
- new net: C2.2, R2.2, U1.3 (+)
- new net: C1.2, ImpactTone1.1, R1.2
Other:
- moved on the sheet: C5, D3, R1, ShellVolume1

Commit message: trying to get simulation to work
Parts:
- added R22: 2K, symbol Device:R
- added R23: 20k, symbol Device:R
- R21: value 56k -> 10k
Connections:
- net GND: now also R22.2
- net at Q2.1 (E), Sweep1.3: now also R23.2; no longer Q3.1 (E)
- net at R16.2, U2.4 (-): now also R22.1
- new net: Q3.1 (E), R23.1
Other:
- moved on the sheet: C10
