File: bass#.kicad_sch (KiCad schematic)
At the start: 57 parts, among them J1 Trigger, J2 CV, J3 Output, Q1 2N3904, Q2 2N3904, Q3 2N3906, Q4 2N3906, U1 TL072, U2 LM13700

Commit message: work on air
Parts:
- C1, C2, C3: footprint (none) -> Capacitor_SMD:C_0603_1608Metric
- D1, D2, D4, D5, D6: footprint (none) -> Diode_SMD:D_0603_1608Metric
- D3: footprint (none) -> LED_SMD:LED_0603_1608Metric
- R1, R10, R11, R12, R13, R14, R2, R3, R4, R5, R6, R7, R8, R9: footprint (none) -> Resistor_SMD:R_0603_1608Metric
- R15: renamed from R23; footprint (none) -> Resistor_SMD:R_0603_1608Metric
- R16: renamed from R22; footprint (none) -> Resistor_SMD:R_0603_1608Metric
- R17: renamed from R15; footprint (none) -> Resistor_SMD:R_0603_1608Metric
- R18: renamed from R16; footprint (none) -> Resistor_SMD:R_0603_1608Metric
- R19: renamed from R17; footprint (none) -> Resistor_SMD:R_0603_1608Metric
- R20: renamed from R18; footprint (none) -> Resistor_SMD:R_0603_1608Metric
- R21: renamed from R19; footprint (none) -> Resistor_SMD:R_0603_1608Metric
- R22: renamed from R20; footprint (none) -> Resistor_SMD:R_0603_1608Metric
- R23: renamed from R21; footprint (none) -> Resistor_SMD:R_0603_1608Metric
- U1: footprint (none) -> Package_SO:SOIC-8_3.9x4.9mm_P1.27mm
- U2: footprint (none) -> Package_SO:SOIC-16_3.9x9.9mm_P1.27mm
Connections:
- net Output: now reaches C7.2, J3.T
