File: power.kicad_sch (KiCad schematic)
At the start: 9 parts, among them J2 Eurorack PWR, U1 TL072, U2 LM13700

Commit message: trying simulation
Parts:
- renumbered C5 to C12, C6 to C13, C7 to C14, C8 to C15, C9 to C16, C10 to C17, J2 to J4
Changed lines of the file:
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@@
+	(wire
+		(pts
+			(xy 133.35 46.99) (xy 125.73 46.99)
+		)
+		(stroke
+			(width 0)
+			(type default)
+		)
+	)
 	(wire
 		(pts
@@
 	(symbol
 		(lib_id "power:PWR_FLAG")
-		(at 125.73 46.99 270)
+		(at 133.35 46.99 270)
 		(unit 1)
 		(exclude_from_sim no)
@@
 		(dnp no)
 		(fields_autoplaced yes)
-		(property "Reference" "#FLG03"
-			(at 127.635 46.99 0)
+		(property "Reference" "#FLG01"
+			(at 135.255 46.99 0)
 			(effects
 				(font
@@
 		)
 		(property "Value" "PWR_FLAG"
-			(at 129.54 46.9899 90)
-			(effects
-				(font
-					(size 1.27 1.27)
-				)
-				(justify left)
-			)
-		)
-		(property "Footprint" ""
-			(at 125.73 46.99 0)
+			(at 137.16 46.9899 90)
+			(effects
+				(font
+					(size 1.27 1.27)
+				)
+				(justify left)
+			)
+		)
+		(property "Footprint" ""
+			(at 133.35 46.99 0)
 			(effects
 				(font
@@
 		)
 		(property "Datasheet" "~"
-			(at 125.73 46.99 0)
+			(at 133.35 46.99 0)
 			(effects
 				(font
@@
 		)
 		(property "Description" "Special symbol for telling ERC where power comes from"
-			(at 125.73 46.99 0)
-			(effects
-				(font
-					(size 1.27 1.27)
-				)
-				(hide yes)
-			)
-		)
-		(pin "1"
-		)
-		(instances
-			(project "bass#"
-				(path "/910cbb2e-c859-40f6-ada9-839bed89c71a/45337cce-6177-4459-9bd9-77e1c110860d"
-					(reference "#FLG03")
+			(at 133.35 46.99 0)
+			(effects
+				(font
+					(size 1.27 1.27)
+				)
+				(hide yes)
+			)
+		)
+		(pin "1"
+		)
+		(instances
+			(project "bass#"
+				(path "/910cbb2e-c859-40f6-ada9-839bed89c71a/45337cce-6177-4459-9bd9-77e1c110860d"
+					(reference "#FLG01")
 					(unit 1)
 				)
@@
 		(dnp no)
 		(fields_autoplaced yes)
-		(property "Reference" "J2"
+		(property "Reference" "J4"
 			(at 59.69 35.56 0)
 			(effects
@@
 			(project "bass#"
 				(path "/910cbb2e-c859-40f6-ada9-839bed89c71a/45337cce-6177-4459-9bd9-77e1c110860d"
-					(reference "J2")
+					(reference "J4")
 					(unit 1)
 				)
@@
 		(on_board yes)
 		(dnp no)
-		(property "Reference" "#PWR014"
+		(property "Reference" "#PWR030"
 			(at 43.18 54.61 0)
 			(effects
@@
 			(project "bass#"
 				(path "/910cbb2e-c859-40f6-ada9-839bed89c71a/45337cce-6177-4459-9bd9-77e1c110860d"
-					(reference "#PWR014")
+					(reference "#PWR030")
 					(unit 1)
 				)
@@
 		(at 86.36 53.34 0)
 		(unit 1)
-		(exclude_from_sim yes)
+		(exclude_from_sim no)
 		(in_bom yes)
 		(on_board yes)
 		(dnp no)
 		(fields_autoplaced yes)
-		(property "Reference" "C6"
+		(property "Reference" "C13"
 			(at 90.17 51.1809 0)
 			(effects
@@
 			(project "bass#"
 				(path "/910cbb2e-c859-40f6-ada9-839bed89c71a/45337cce-6177-4459-9bd9-77e1c110860d"
-					(reference "C6")
+					(reference "C13")
 					(unit 1)
 				)
@@
 		(dnp no)
 		(fields_autoplaced yes)
-		(property "Reference" "C7"
+		(property "Reference" "C14"
 			(at 110.49 36.8299 0)
 			(effects
@@
 			(project "bass#"
 				(path "/910cbb2e-c859-40f6-ada9-839bed89c71a/45337cce-6177-4459-9bd9-77e1c110860d"
-					(reference "C7")
+					(reference "C14")
 					(unit 1)
 				)
@@
 		(dnp no)
 		(fields_autoplaced yes)
-		(property "Reference" "#PWR013"
+		(property "Reference" "#PWR032"
 			(at 59.69 54.61 0)
 			(effects
@@
 			(project "bass#"
 				(path "/910cbb2e-c859-40f6-ada9-839bed89c71a/45337cce-6177-4459-9bd9-77e1c110860d"
-					(reference "#PWR013")
+					(reference "#PWR032")
 					(unit 1)
 				)
@@
 		(dnp no)
 		(fields_autoplaced yes)
-		(property "Reference" "#FLG02"
+		(property "Reference" "#FLG03"
 			(at 166.37 60.325 0)
 			(effects
@@
 			(project "bass#"
 				(path "/910cbb2e-c859-40f6-ada9-839bed89c71a/45337cce-6177-4459-9bd9-77e1c110860d"
-					(reference "#FLG02")
+					(reference "#FLG03")
 					(unit 1)
 				)
@@
 		(dnp no)
 		(fields_autoplaced yes)
-		(property "Reference" "#PWR012"
+		(property "Reference" "#PWR031"
 			(at 59.69 35.56 0)
 			(effects
@@
 			(project "bass#"
 				(path "/910cbb2e-c859-40f6-ada9-839bed89c71a/45337cce-6177-4459-9bd9-77e1c110860d"
-					(reference "#PWR012")
+					(reference "#PWR031")
 					(unit 1)
 				)
@@
 		(dnp no)
 		(fields_autoplaced yes)
-		(property "Reference" "#FLG01"
+		(property "Reference" "#FLG02"
 			(at 166.37 32.385 0)
 			(effects
@@
 			(project "bass#"
 				(path "/910cbb2e-c859-40f6-ada9-839bed89c71a/45337cce-6177-4459-9bd9-77e1c110860d"
-					(reference "#FLG01")
+					(reference "#FLG02")
 					(unit 1)
 				)
@@
 		(on_board yes)
 		(dnp no)
-		(property "Reference" "#PWR011"
+		(property "Reference" "#PWR033"
 			(at 74.93 54.61 0)
 			(effects
@@
 			(project "bass#"
 				(path "/910cbb2e-c859-40f6-ada9-839bed89c71a/45337cce-6177-4459-9bd9-77e1c110860d"
-					(reference "#PWR011")
+					(reference "#PWR033")
 					(unit 1)
 				)
@@
 		(at 86.36 38.1 0)
 		(unit 1)
-		(exclude_from_sim yes)
+		(exclude_from_sim no)
 		(in_bom yes)
 		(on_board yes)
 		(dnp no)
 		(fields_autoplaced yes)
-		(property "Reference" "C5"
+		(property "Reference" "C12"
 			(at 90.17 35.9409 0)
 			(effects
@@
 			(project "bass#"
 				(path "/910cbb2e-c859-40f6-ada9-839bed89c71a/45337cce-6177-4459-9bd9-77e1c110860d"
-					(reference "C5")
+					(reference "C12")
 					(unit 1)
 				)
@@
 		(at 125.73 38.1 0)
 		(unit 1)
-		(exclude_from_sim yes)
+		(exclude_from_sim no)
 		(in_bom yes)
 		(on_board yes)
 		(dnp no)
 		(fields_autoplaced yes)
-		(property "Reference" "C9"
+		(property "Reference" "C16"
 			(at 129.54 36.8299 0)
 			(effects
@@
 			(project "bass#"
 				(path "/910cbb2e-c859-40f6-ada9-839bed89c71a/45337cce-6177-4459-9bd9-77e1c110860d"
-					(reference "C9")
+					(reference "C16")
 					(unit 1)
 				)
@@
 		(at 125.73 53.34 0)
 		(unit 1)
-		(exclude_from_sim yes)
+		(exclude_from_sim no)
 		(in_bom yes)
 		(on_board yes)
 		(dnp no)
 		(fields_autoplaced yes)
-		(property "Reference" "C10"
+		(property "Reference" "C17"
 			(at 129.54 52.0699 0)
 			(effects
@@
 			(project "bass#"
 				(path "/910cbb2e-c859-40f6-ada9-839bed89c71a/45337cce-6177-4459-9bd9-77e1c110860d"
-					(reference "C10")
+					(reference "C17")
 					(unit 1)
 				)
@@
 		(dnp no)
 		(fields_autoplaced yes)
-		(property "Reference" "C8"
+		(property "Reference" "C15"
 			(at 110.49 52.0699 0)
 			(effects
@@
 			(project "bass#"
 				(path "/910cbb2e-c859-40f6-ada9-839bed89c71a/45337cce-6177-4459-9bd9-77e1c110860d"
-					(reference "C8")
+					(reference "C15")
 					(unit 1)
 				)
