File: power.kicad_sch (KiCad schematic)
At the start: 9 parts, among them J4 Eurorack PWR, U1 TL072, U2 LM13700

Commit message: work on air
Parts:
- C12, C13: footprint (none) -> Capacitor_SMD:CP_Elec_4x3
- C14, C15, C16, C17: footprint (none) -> Capacitor_SMD:C_0603_1608Metric
- U1: footprint (none) -> Package_SO:SOIC-8_3.9x4.9mm_P1.27mm
- U2: footprint (none) -> Package_SO:SOIC-16_3.9x9.9mm_P1.27mm
Changed lines of the file:
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@@
 		(on_board yes)
 		(dnp no)
-		(property "Reference" "#PWR030"
+		(property "Reference" "#PWR031"
 			(at 43.18 54.61 0)
 			(effects
@@
 			(project "bass#"
 				(path "/910cbb2e-c859-40f6-ada9-839bed89c71a/45337cce-6177-4459-9bd9-77e1c110860d"
-					(reference "#PWR030")
+					(reference "#PWR031")
 					(unit 1)
 				)
@@
 			)
 		)
-		(property "Footprint" ""
+		(property "Footprint" "Capacitor_SMD:CP_Elec_4x3"
 			(at 87.3252 57.15 0)
 			(effects
@@
 			)
 		)
-		(property "Footprint" ""
+		(property "Footprint" "Capacitor_SMD:C_0603_1608Metric"
 			(at 107.6452 41.91 0)
 			(effects
@@
 		(dnp no)
 		(fields_autoplaced yes)
-		(property "Reference" "#PWR032"
+		(property "Reference" "#PWR033"
 			(at 59.69 54.61 0)
 			(effects
@@
 			(project "bass#"
 				(path "/910cbb2e-c859-40f6-ada9-839bed89c71a/45337cce-6177-4459-9bd9-77e1c110860d"
-					(reference "#PWR032")
+					(reference "#PWR033")
 					(unit 1)
 				)
@@
 		(dnp no)
 		(fields_autoplaced yes)
-		(property "Reference" "#PWR031"
+		(property "Reference" "#PWR032"
 			(at 59.69 35.56 0)
 			(effects
@@
 			(project "bass#"
 				(path "/910cbb2e-c859-40f6-ada9-839bed89c71a/45337cce-6177-4459-9bd9-77e1c110860d"
-					(reference "#PWR031")
+					(reference "#PWR032")
 					(unit 1)
 				)
@@
 		(on_board yes)
 		(dnp no)
-		(property "Reference" "#PWR033"
+		(property "Reference" "#PWR034"
 			(at 74.93 54.61 0)
 			(effects
@@
 			(project "bass#"
 				(path "/910cbb2e-c859-40f6-ada9-839bed89c71a/45337cce-6177-4459-9bd9-77e1c110860d"
-					(reference "#PWR033")
+					(reference "#PWR034")
 					(unit 1)
 				)
@@
 			)
 		)
-		(property "Footprint" ""
+		(property "Footprint" "Package_SO:SOIC-8_3.9x4.9mm_P1.27mm"
 			(at 154.94 46.99 0)
 			(effects
@@
 			)
 		)
-		(property "Footprint" ""
+		(property "Footprint" "Package_SO:SOIC-16_3.9x9.9mm_P1.27mm"
 			(at 161.29 46.355 0)
 			(effects
@@
 			)
 		)
-		(property "Footprint" ""
+		(property "Footprint" "Capacitor_SMD:CP_Elec_4x3"
 			(at 87.3252 41.91 0)
 			(effects
@@
 			)
 		)
-		(property "Footprint" ""
+		(property "Footprint" "Capacitor_SMD:C_0603_1608Metric"
 			(at 126.6952 41.91 0)
 			(effects
@@
 			)
 		)
-		(property "Footprint" ""
+		(property "Footprint" "Capacitor_SMD:C_0603_1608Metric"
 			(at 126.6952 57.15 0)
 			(effects
@@
 			)
 		)
-		(property "Footprint" ""
+		(property "Footprint" "Capacitor_SMD:C_0603_1608Metric"
 			(at 107.6452 57.15 0)
 			(effects
