File: simulation.kicad_sch (KiCad schematic)
At the start: 3 parts

Commit message: trying simulation
Connections:
- net GND renamed 0
Other:
- moved on the sheet: V2, V3
Changed lines of the file:
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@@
 	)
 	(junction
-		(at 128.27 45.72)
+		(at 36.83 97.79)
 		(diameter 0)
 		(color 0 0 0 0)
 	)
+	(junction
+		(at 41.91 97.79)
+		(diameter 0)
+		(color 0 0 0 0)
+	)
 	(wire
 		(pts
-			(xy 128.27 41.91) (xy 128.27 45.72)
+			(xy 41.91 93.98) (xy 41.91 97.79)
 		)
 		(stroke
@@
 	(wire
 		(pts
-			(xy 128.27 45.72) (xy 128.27 48.26)
+			(xy 41.91 97.79) (xy 41.91 100.33)
 		)
 		(stroke
@@
 	(wire
 		(pts
-			(xy 119.38 45.72) (xy 128.27 45.72)
+			(xy 33.02 97.79) (xy 36.83 97.79)
 		)
 		(stroke
@@
 	(wire
 		(pts
-			(xy 34.29 34.29) (xy 36.83 34.29)
+			(xy 36.83 97.79) (xy 41.91 97.79)
 		)
 		(stroke
@@
 	(wire
 		(pts
-			(xy 34.29 41.91) (xy 34.29 34.29)
+			(xy 30.48 88.9) (xy 36.83 88.9)
 		)
 		(stroke
@@
 		)
 	)
+	(wire
+		(pts
+			(xy 36.83 88.9) (xy 36.83 97.79)
+		)
+		(stroke
+			(width 0)
+			(type default)
+		)
+	)
+	(wire
+		(pts
+			(xy 34.29 34.29) (xy 36.83 34.29)
+		)
+		(stroke
+			(width 0)
+			(type default)
+		)
+	)
+	(wire
+		(pts
+			(xy 34.29 41.91) (xy 34.29 34.29)
+		)
+		(stroke
+			(width 0)
+			(type default)
+		)
+	)
 	(global_label "TrigIn"
 		(shape output)
@@
 	(symbol
 		(lib_id "power:-12V")
-		(at 128.27 58.42 180)
+		(at 41.91 110.49 180)
 		(unit 1)
 		(exclude_from_sim no)
@@
 		(dnp no)
 		(fields_autoplaced yes)
-		(property "Reference" "#PWR035"
-			(at 128.27 54.61 0)
+		(property "Reference" "#PWR037"
+			(at 41.91 106.68 0)
 			(effects
 				(font
@@
 		)
 		(property "Value" "-12V"
-			(at 128.27 63.5 0)
+			(at 41.91 115.57 0)
 			(effects
 				(font
@@
 		)
 		(property "Footprint" ""
-			(at 128.27 58.42 0)
+			(at 41.91 110.49 0)
 			(effects
 				(font
@@
 		)
 		(property "Datasheet" ""
-			(at 128.27 58.42 0)
+			(at 41.91 110.49 0)
 			(effects
 				(font
@@
 		)
 		(property "Description" "Power symbol creates a global label with name \"-12V\""
-			(at 128.27 58.42 0)
+			(at 41.91 110.49 0)
 			(effects
 				(font
@@
 			(project ""
 				(path "/910cbb2e-c859-40f6-ada9-839bed89c71a/ed78e2ce-4e0d-40b3-9111-86efba882b34"
-					(reference "#PWR035")
+					(reference "#PWR037")
 					(unit 1)
 				)
@@
 			)
 		)
-		(property "Sim.Params" "y1=0 y2=5 td=2n tr=2n tf=2n tw=50n per=100n"
+		(property "Sim.Params" "y1=0 y2=5 td=2n tr=2n tf=2n tw=4m per=700m"
 			(at 38.1 49.4001 0)
 			(effects
@@
 	(symbol
 		(lib_id "Simulation_SPICE:VDC")
-		(at 128.27 36.83 0)
+		(at 41.91 88.9 0)
 		(unit 1)
 		(exclude_from_sim no)
@@
 		(fields_autoplaced yes)
 		(property "Reference" "V2"
-			(at 132.08 35.4301 0)
+			(at 45.72 87.5001 0)
 			(effects
 				(font
@@
 		)
 		(property "Value" "12"
-			(at 132.08 37.9701 0)
+			(at 45.72 90.0401 0)
 			(effects
 				(font
@@
 		)
 		(property "Footprint" ""
-			(at 128.27 36.83 0)
+			(at 41.91 88.9 0)
 			(effects
 				(font
@@
 		)
 		(property "Datasheet" "https://ngspice.sourceforge.io/docs/ngspice-html-manual/manual.xhtml#sec_Independent_Sources_for"
-			(at 128.27 36.83 0)
+			(at 41.91 88.9 0)
 			(effects
 				(font
@@
 		)
 		(property "Description" "Voltage source, DC"
-			(at 128.27 36.83 0)
+			(at 41.91 88.9 0)
 			(effects
 				(font
@@
 		)
 		(property "Sim.Pins" "1=+ 2=-"
-			(at 128.27 36.83 0)
+			(at 41.91 88.9 0)
 			(effects
 				(font
@@
 		)
 		(property "Sim.Type" "DC"
-			(at 128.27 36.83 0)
+			(at 41.91 88.9 0)
 			(effects
 				(font
@@
 		)
 		(property "Sim.Device" "V"
-			(at 128.27 36.83 0)
+			(at 41.91 88.9 0)
 			(effects
 				(font
@@
 	)
 	(symbol
-		(lib_id "power:GND")
-		(at 119.38 45.72 0)
+		(lib_id "Simulation_SPICE:0")
+		(at 30.48 88.9 0)
 		(unit 1)
 		(exclude_from_sim no)
@@
 		(dnp no)
 		(fields_autoplaced yes)
-		(property "Reference" "#PWR037"
-			(at 119.38 52.07 0)
-			(effects
-				(font
-					(size 1.27 1.27)
-				)
-				(hide yes)
-			)
-		)
-		(property "Value" "GND"
-			(at 119.38 50.8 0)
+		(property "Reference" "#GND01"
+			(at 30.48 93.98 0)
+			(effects
+				(font
+					(size 1.27 1.27)
+				)
+				(hide yes)
+			)
+		)
+		(property "Value" "0"
+			(at 30.48 86.36 0)
 			(effects
 				(font
@@
 		)
 		(property "Footprint" ""
-			(at 119.38 45.72 0)
-			(effects
-				(font
-					(size 1.27 1.27)
-				)
-				(hide yes)
-			)
-		)
-		(property "Datasheet" ""
-			(at 119.38 45.72 0)
-			(effects
-				(font
-					(size 1.27 1.27)
-				)
-				(hide yes)
-			)
-		)
-		(property "Description" "Power symbol creates a global label with name \"GND\" , ground"
-			(at 119.38 45.72 0)
+			(at 30.48 88.9 0)
+			(effects
+				(font
+					(size 1.27 1.27)
+				)
+				(hide yes)
+			)
+		)
+		(property "Datasheet" "https://ngspice.sourceforge.io/docs/ngspice-html-manual/manual.xhtml#subsec_Circuit_elements__device"
+			(at 30.48 99.06 0)
+			(effects
+				(font
+					(size 1.27 1.27)
+				)
+				(hide yes)
+			)
+		)
+		(property "Description" "0V reference potential for simulation"
+			(at 30.48 96.52 0)
 			(effects
 				(font
@@
 			(project ""
 				(path "/910cbb2e-c859-40f6-ada9-839bed89c71a/ed78e2ce-4e0d-40b3-9111-86efba882b34"
-					(reference "#PWR037")
+					(reference "#GND01")
+					(unit 1)
+				)
+			)
+		)
+	)
+	(symbol
+		(lib_id "power:GND")
+		(at 33.02 97.79 0)
+		(unit 1)
+		(exclude_from_sim no)
+		(in_bom yes)
+		(on_board yes)
+		(dnp no)
+		(fields_autoplaced yes)
+		(property "Reference" "#PWR034"
+			(at 33.02 104.14 0)
+			(effects
+				(font
+					(size 1.27 1.27)
+				)
+				(hide yes)
+			)
+		)
+		(property "Value" "GND"
+			(at 33.02 102.87 0)
+			(effects
+				(font
+					(size 1.27 1.27)
+				)
+			)
+		)
+		(property "Footprint" ""
+			(at 33.02 97.79 0)
+			(effects
+				(font
+					(size 1.27 1.27)
+				)
+				(hide yes)
+			)
+		)
+		(property "Datasheet" ""
+			(at 33.02 97.79 0)
+			(effects
+				(font
+					(size 1.27 1.27)
+				)
+				(hide yes)
+			)
+		)
+		(property "Description" "Power symbol creates a global label with name \"GND\" , ground"
+			(at 33.02 97.79 0)
+			(effects
+				(font
+					(size 1.27 1.27)
+				)
+				(hide yes)
+			)
+		)
+		(pin "1"
+		)
+		(instances
+			(project ""
+				(path "/910cbb2e-c859-40f6-ada9-839bed89c71a/ed78e2ce-4e0d-40b3-9111-86efba882b34"
+					(reference "#PWR034")
 					(unit 1)
 				)
@@
 	(symbol
 		(lib_id "Simulation_SPICE:VDC")
-		(at 128.27 53.34 0)
+		(at 41.91 105.41 0)
 		(unit 1)
 		(exclude_from_sim no)
@@
 		(fields_autoplaced yes)
 		(property "Reference" "V3"
-			(at 132.08 51.9401 0)
+			(at 45.72 104.0101 0)
 			(effects
 				(font
@@
 		)
 		(property "Value" "12"
-			(at 132.08 54.4801 0)
+			(at 45.72 106.5501 0)
 			(effects
 				(font
@@
 		)
 		(property "Footprint" ""
-			(at 128.27 53.34 0)
+			(at 41.91 105.41 0)
 			(effects
 				(font
@@
 		)
 		(property "Datasheet" "https://ngspice.sourceforge.io/docs/ngspice-html-manual/manual.xhtml#sec_Independent_Sources_for"
-			(at 128.27 53.34 0)
+			(at 41.91 105.41 0)
 			(effects
 				(font
@@
 		)
 		(property "Description" "Voltage source, DC"
-			(at 128.27 53.34 0)
+			(at 41.91 105.41 0)
 			(effects
 				(font
@@
 		)
 		(property "Sim.Pins" "1=+ 2=-"
-			(at 128.27 53.34 0)
+			(at 41.91 105.41 0)
 			(effects
 				(font
@@
 		)
 		(property "Sim.Type" "DC"
-			(at 128.27 53.34 0)
+			(at 41.91 105.41 0)
 			(effects
 				(font
@@
 		)
 		(property "Sim.Device" "V"
-			(at 128.27 53.34 0)
+			(at 41.91 105.41 0)
 			(effects
 				(font
@@
 		(dnp no)
 		(fields_autoplaced yes)
-		(property "Reference" "#PWR034"
+		(property "Reference" "#PWR035"
 			(at 34.29 58.42 0)
 			(effects
@@
 			(project ""
 				(path "/910cbb2e-c859-40f6-ada9-839bed89c71a/ed78e2ce-4e0d-40b3-9111-86efba882b34"
-					(reference "#PWR034")
+					(reference "#PWR035")
 					(unit 1)
 				)
@@
 	(symbol
 		(lib_id "power:+12V")
-		(at 128.27 31.75 0)
+		(at 41.91 83.82 0)
 		(unit 1)
 		(exclude_from_sim no)
@@
 		(fields_autoplaced yes)
 		(property "Reference" "#PWR036"
-			(at 128.27 35.56 0)
+			(at 41.91 87.63 0)
 			(effects
 				(font
@@
 		)
 		(property "Value" "+12V"
-			(at 128.27 26.67 0)
+			(at 41.91 78.74 0)
 			(effects
 				(font
@@
 		)
 		(property "Footprint" ""
-			(at 128.27 31.75 0)
+			(at 41.91 83.82 0)
 			(effects
 				(font
@@
 		)
 		(property "Datasheet" ""
-			(at 128.27 31.75 0)
+			(at 41.91 83.82 0)
 			(effects
 				(font
@@
 		)
 		(property "Description" "Power symbol creates a global label with name \"+12V\""
-			(at 128.27 31.75 0)
-			(effects
-				(font
+			(at 41.91 83.82 0)
+			(effects
+				(font
