File: simulation.kicad_sch (KiCad schematic)
At the start: 3 parts

Commit message: work on air
Other:
- note added: ".control set controlswait linearize v(Output) * file, sample rate, format, multiplier, offset, oversampling sndparam /Users/viktor/dev/ee/bass#/out-from-simulation.wav 48000 wav32 3.5 0.0 2 sndprint v(Output) rusage .endc"
